Commit message: Actually publish camera info correctly

File: prius_description/urdf/prius.urdf (robot description, URDF)
Before this commit: robot prius, 24 links, 23 joints
Links:
- added link front_camera_ros_link
Joints:
- added joint front_camera_ros_joint: type fixed, parent front_camera_link, child front_camera_ros_link, origin xyz=0 0.0 0.0 rpy=-1.5707963267948966 0.0 -1.5707963267948966

Commit message: Sensor settings for prius and more stuff in the simulation

File: prius_description/urdf/prius.urdf (robot description, URDF)
Before this commit: robot prius, 25 links, 24 joints
Links:
- added link imu_link, mass 1
Joints:
- added joint imu_joint: type fixed, parent chassis, child imu_link, origin xyz=0 1.45 0.4 rpy=0 0 -1.57
