Commit message: incorporated model of RCV

File: rcv_description/urdf/rcv.urdf (robot description, URDF)
Before this commit: robot rcv, 9 links, 8 joints
Links:
- added link rl_axle, mass 1
- added link rr_axle, mass 1
- link chassis: mass 1356.0 -> 400.0; geometry collision box size=1.279154 0.625988 0.171868; collision box size=1.285130 0.771189 0.226557
- link front_left_wheel: mass 11 -> 25
- link front_right_wheel: mass 11 -> 25
- link rear_left_wheel: mass 11 -> 25
- link rear_right_wheel: mass 11 -> 25
Joints:
- added joint rear_left_steer_joint: type continuous, parent chassis, child rl_axle, origin xyz=0.75 1.0 0.3 rpy=0 0 0, axis 0 0 1, limit lower=-0.8727 upper=0.8727 effort=10000000 velocity=1000000
- added joint rear_right_steer_joint: type continuous, parent chassis, child rr_axle, origin xyz=-0.75 1.0 0.3 rpy=0 0 0, axis 0 0 1, limit lower=-0.8727 upper=0.8727 effort=10000000 velocity=1000000
- joint front_left_steer_joint: origin xyz=0.767 -1.41 0.3 rpy=0 0 0 -> xyz=0.75 -1.0 0.3 rpy=0 0 0
- joint front_right_steer_joint: origin xyz=-0.767 -1.41 0.3 rpy=0 0 0 -> xyz=-0.75 -1.0 0.3 rpy=0 0 0
- joint rear_left_wheel_joint: origin xyz=0.793 1.45 0.3 rpy=0 0 0 -> xyz=0 0 0 rpy=0 0 0; parent chassis -> rl_axle
- joint rear_right_wheel_joint: origin xyz=-0.793 1.45 0.3 rpy=0 0 0 -> xyz=0 0 0 rpy=0 0 0; parent chassis -> rr_axle
