Commit message: changed baselink origin to geometric center in rcv urdf

File: rcv_gazebo_description/urdf/rcv.urdf (robot description, URDF)
Before this commit: robot rcv, 11 links, 10 joints
Links:
- link chassis: geometry collision box size=1.279154 0.625988 0.171868; collision box size=1.285130 0.771189 0.226557
Joints:
- joint base_link_connection: origin xyz=1.45 0 0 rpy=0 0 1.57 -> xyz=0 0 0 rpy=0 0 1.57

Commit message: changed torque req interpretation from prius to rcv

File: rcv_gazebo_description/urdf/rcv.urdf (robot description, URDF)
Before this commit: robot rcv, 11 links, 10 joints
Links:
- link chassis: geometry collision box size=1.279154 0.625988 0.171868; collision box size=1.285130 0.771189 0.226557
- link front_left_wheel: geometry collision sphere radius=0.31265; visual mesh filename=package://prius_description/meshes/wheel.obj scale=0.0065 0.01 0.01
- link front_right_wheel: geometry collision sphere radius=0.31265; visual mesh filename=package://prius_description/meshes/wheel.obj scale=0.0065 0.01 0.01
- link rear_left_wheel: geometry collision sphere radius=0.31265; visual mesh filename=package://prius_description/meshes/wheel.obj scale=0.0065 0.01 0.01
- link rear_right_wheel: geometry collision sphere radius=0.31265; visual mesh filename=package://prius_description/meshes/wheel.obj scale=0.0065 0.01 0.01
- link steering_wheel: geometry visual mesh filename=package://prius_description/meshes/steering_wheel.obj scale=0.007 0.007 0.007
Joints:
- joint front_left_steer_joint: origin xyz=0.75 -1.0 0.3 rpy=0 0 0 -> xyz=0.75 -1.0 0.16 rpy=0 0 0
- joint front_right_steer_joint: origin xyz=-0.75 -1.0 0.3 rpy=0 0 0 -> xyz=-0.75 -1.0 0.16 rpy=0 0 0
- joint rear_left_steer_joint: origin xyz=0.75 1.0 0.3 rpy=0 0 0 -> xyz=0.75 1.0 0.16 rpy=0 0 0
- joint rear_right_steer_joint: origin xyz=-0.75 1.0 0.3 rpy=0 0 0 -> xyz=-0.75 1.0 0.16 rpy=0 0 0
- joint steering_joint: origin xyz=0.357734 -0.627868 0.988243 rpy=-1.302101 0 0 -> xyz=0.275 -0.12 0.63 rpy=-1.302101 0 0
